Commit message: simulation model

File: src/urdf/al5d.urdf (robot description, URDF)
Before this commit: robot AL5D, 5 links, 4 joints
Links:
- link link1: geometry visual box size=0.06 0.05 0.030; visual cylinder length=0.01 radius=0.045
- link link2: geometry visual box size=0.105 0.06 0.026; visual cylinder length=0.06 radius=0.013
- link link3: geometry visual box size=0.06 0.05 0.028; visual box size=0.06 0.05 0.028
- link link4: geometry visual box size=0.03 0.06 0.026; visual box size=0.0375 0.013 0.022
Joints:
- joint joint1: limit lower=-2.61 upper=2.61 effort=0.5 velocity=6.0 -> lower=0 upper=3.1415 effort=0.5 velocity=6.0
- joint joint2: axis 1 0 0 -> 0 -1 0; limit lower=-1.75 upper=1.75 effort=0.5 velocity=6.0 -> lower=0 upper=3.1415 effort=0.5 velocity=6.0; origin xyz=0 0.015 0.027 rpy=0 0 0 -> xyz=0.015 0 0.027 rpy=0 0 0
- joint joint3: axis -1 0 0 -> 0 1 0; limit lower=-2.55 upper=2.55 effort=0.5 velocity=6.0 -> lower=-1.5708 upper=1.5708 effort=0.5 velocity=6.0; origin xyz=0 0 0.105 rpy=0 0 0 -> xyz=0.105 0 0 rpy=0 0 0
- joint joint4: axis 1 0 0 -> 0 1 0; limit lower=-1.80 upper=1.80 effort=0.5 velocity=6.0 -> lower=-1.5708 upper=1.5708 effort=0.5 velocity=6.0; origin xyz=0 0 0.120 rpy=0 0 0 -> xyz=0.120 0 0 rpy=0 0 0

File: src/urdf/al5d_old.urdf (robot description, URDF)
Before this commit: robot AL5D, 5 links, 4 joints
Links:
- link base_link: geometry visual box size=0.09 0.1 0.024; visual cylinder length=0.040 radius=0.045
- link link1: geometry visual box size=0.05 0.06 0.030; visual cylinder length=0.01 radius=0.045
- link link2: geometry visual box size=0.06 0.026 0.105; visual cylinder length=0.06 radius=0.013
- link link3: geometry visual box size=0.05 0.028 0.06; visual box size=0.05 0.028 0.06
- link link4: geometry visual box size=0.013 0.022 0.0375; visual box size=0.013 0.022 0.0375
Joints:
- joint joint2: axis 0 1 0 -> 1 0 0; origin xyz=0.015 0 0.027 rpy=0 0 0 -> xyz=0 0.015 0.027 rpy=0 0 0
- joint joint3: axis 0 -1 0 -> -1 0 0
- joint joint4: axis 0 1 0 -> 1 0 0

Commit message: final day

File: src/urdf/al5d.urdf (robot description, URDF)
Before this commit: robot AL5D, 5 links, 4 joints
Joints:
- joint joint3: axis 0 1 0 -> 0 -1 0
- joint joint4: axis 0 1 0 -> 0 -1 0
